Commit message: Implement ros2 control gazebo

File: description/lidar.xacro (robot description, xacro)
@@ -18,7 +18,7 @@
 			</geometry>
 		</collision>
-		<inertial_cylinder mass="0.1" length="0.04" radius="0.05">
+		<xacro:inertial_cylinder mass="0.1" length="0.04" radius="0.05">
 			<origin xyz="0 0 0" rpy="0 0 0" />
-		</inertial_cylinder>
+		</xacro:inertial_cylinder>
 	</link>
 	<gazebo reference="laser_frame">

File: description/robot.urdf.xacro (robot description, xacro)
@@ -1,7 +1,7 @@
 <?xml version="1.0"?>
 <robot xmlns:xacro="http://www.ros.org/wiki/xacro" name="robot">
-	<include filename="robot_core.xacro" />
-	<!-- <include filename="gazebo_control.xacro" /> -->
-	<include filename="lidar.xacro" />
-	<include filename="ros2_control.xacro" />
+	<xacro:include filename="robot_core.xacro" />
+	<!-- <xacro:include filename="gazebo_control.xacro" />  -->
+	<xacro:include filename="lidar.xacro" />
+	<xacro:include filename="ros2_control.xacro" />
 </robot>

File: description/robot_core.xacro (robot description, xacro)
@@ -1,5 +1,5 @@
 <?xml version="1.0"?>
 <robot xmlns:xacro="http://www.ros.org/wiki/xacro">
-	<include filename="inertial_macros.xacro" />
+	<xacro:include filename="inertial_macros.xacro" />
 	<material name="white">
 		<color rgba="1 1 1 1" />
@@ -37,7 +37,7 @@
 			</geometry>
 		</collision>
-		<inertial_box mass="0.5" x="0.25" y="0.25" z="0.12">
+		<xacro:inertial_box mass="0.5" x="0.25" y="0.25" z="0.12">
 			<origin xyz="0 0 0.03915" rpy="0 0 0" />
-		</inertial_box>
+		</xacro:inertial_box>
 	</link>
 	<gazebo reference="chassis">
@@ -65,7 +65,7 @@
 			</geometry>
 		</collision>
-		<inertial_cylinder mass="0.1" length="0.01" radius="0.045">
+		<xacro:inertial_cylinder mass="0.1" length="0.01" radius="0.045">
 			<origin xyz="0 0 0" rpy="0 0 0" />
-		</inertial_cylinder>
+		</xacro:inertial_cylinder>
 	</link>
 	<gazebo reference="left_wheel">
@@ -93,7 +93,7 @@
 			</geometry>
 		</collision>
-		<inertial_cylinder mass="0.1" length="0.01" radius="0.045">
+		<xacro:inertial_cylinder mass="0.1" length="0.01" radius="0.045">
 			<origin xyz="0 0 0" rpy="0 0 0" />
-		</inertial_cylinder>
+		</xacro:inertial_cylinder>
 	</link>
 	<gazebo reference="right_wheel">
@@ -120,18 +120,7 @@
 			</geometry>
 		</collision>
-<<<<<<< HEAD
-		<inertial_sphere mass="0.1" radius="0.02415">
-			<origin xyz="0 0 0" rpy="0 0 0" />
-		</inertial_sphere>
-=======
 		<xacro:inertial_sphere mass="0.1" radius="0.02415">
 			<origin xyz="0 0 0" rpy="0 0 0"/>
 		</xacro:inertial_sphere>
-		<gazebo reference="front                _caster_wheel">
-			<material>Gazebo/Black</material>
-			<mu1 value="0.001"/>
-			<mu2 value="0.001"/>
-		</gazebo>
->>>>>>> d0f761d1e2e5992d1c0384035b248e425c0e06f5
 	</link>
 	<gazebo reference="front_caster_wheel">
@@ -160,7 +149,7 @@
 			</geometry>
 		</collision>
-		<inertial_sphere mass="0.1" radius="0.02415">
-			<origin xyz="0 0 0" rpy="0 0 0" />
-		</inertial_sphere>
+		<xacro:inertial_sphere mass="0.1" radius="0.02415">
+			<origin xyz="0 0 0" rpy="0 0 0"/>
+		</xacro:inertial_sphere>
 	</link>
 	<gazebo reference="back_caster_wheel">
@@ -172,3 +161,2 @@
 	</gazebo>
 </robot>
-0

File: description/ros2_control.xacro (robot description, xacro)
@@ -1,41 +1,29 @@
 <?xml version="1.0"?>
-<robot xmlns:xacro="http://www.ros.org/wiki/xacro" name="robot">
-	<ros2_control name="GazeboSystem" type="system">
-		<hardware>
-			<plugin>
-				gazebo_ros2_control/GazeboSystem
-			</plugin>
-		</hardware>
-		<joint name="left_wheel_joint">
-			<command_interface name="velocity">
-				<param name="min">
-					-10
-				</param>
-				<param name="max">
-					10
-				</param>
-			</command_interface>
-			<state_interface name="position" />
-			<state_interface name="velocity" />
-		</joint>
-		<joint name="right_wheel_joint">
-			<command_interface name="velocity">
-				<param name="min">
-					-10
-				</param>
-				<param name="max">
-					10
-				</param>
-			</command_interface>
-			<state_interface name="velocity" />
-			<state_interface name="position" />
-		</joint>
-	</ros2_control>
-	<gazebo>
-		<plugin filename="libgazebo_ros2_control.so" name="gazebo_ros2_control">
-			<parameters>
-				$(find wubot)/config/my_controllers.yaml
-			</parameters>
-		</plugin>
-	</gazebo>
+<robot xmlns:xacro="http://www.ros.org/wiki/xacro">
+    <ros2_control name="GazeboSystem" type="system">
+        <hardware>
+            <plugin>gazebo_ros2_control/GazeboSystem</plugin>
+        </hardware>
+        <joint name="left_wheel_joint">
+            <command_interface name="velocity">
+                <param name="min">-10</param>
+                <param name="max">10</param>
+            </command_interface>
+            <state_interface name="velocity"/>
+            <state_interface name="position"/>
+        </joint>
+        <joint name="right_wheel_joint">
+            <command_interface name="velocity">
+                <param name="min">-10</param>
+                <param name="max">10</param>
+            </command_interface>
+            <state_interface name="velocity"/>
+            <state_interface name="position"/>
+        </joint>
+    </ros2_control>
+    <gazebo>
+        <plugin name="gazebo_ros2_control" filename="libgazebo_ros2_control.so">
+            <parameters>$(find wubot)/config/my_controllers.yaml</parameters>
+        </plugin>
+    </gazebo>
 </robot>

Commit message: Get slam running

File: description/lidar.xacro (robot description, xacro)
@@ -4,5 +4,5 @@
 		<parent link="chassis" />
 		<child link="laser_frame" />
-		<origin xyz="0 0 0.12" rpy="0 0 0" />
+		<origin xyz="0 0 0.12" rpy="0 0 ${pi}" />
 	</joint>
 	<link name="laser_frame">
@@ -19,5 +19,5 @@
 		</collision>
 		<xacro:inertial_cylinder mass="0.1" length="0.04" radius="0.05">
-			<origin xyz="0 0 0" rpy="0 0 0" />
+			<origin xyz="0 0 0" rpy="0 0 ${pi}" />
 		</xacro:inertial_cylinder>
 	</link>

File: description/robot_core.xacro (robot description, xacro)
@@ -17,4 +17,11 @@
 	<link name="base_link">
 	</link>
+	<joint name="base_footprint_joint" type="fixed">
+        <parent link="base_link"/>
+        <child link="base_footprint"/>
+        <origin xyz="0 0 0" rpy="0 0 0"/>
+    </joint>
+    <link name="base_footprint">
+    </link>
 	<!-- CHASSIS -->
 	<joint name="chassis_joint" type="fixed">
