Commit message: Added wheels

File: description/robot_core.xacro (robot description, xacro)
@@ -22,10 +22,38 @@
 	<link name="chassis">
 		<visual>
-		    <origin xyz="0 0 0.02085" rpy="0 0 0"/>
+		    <origin xyz="0 0 0.03915" rpy="0 0 0"/>
 		    <geometry>
-		        <box size="0.25 0.25 0.1"/>
+		        <box size="0.25 0.25 0.12"/>
 		    </geometry>
 		    <material name="white"/>
 		</visual>
 	</link>
+	<joint name="left_wheel_joint" type="continuous">
+		<parent link="base_link"/>
+		<child link="left_wheel"/>
+		<origin xyz="0 0.1375 0" rpy="-${pi/2} 0 0"/>
+		<axis xyz="0 0 1"/>
+	</joint>
+	<link name="left_wheel">
+		<visual>
+			<geometry>
+				<cylinder length="0.01" radius="0.045" />/>
+			</geometry>
+			<material name="blue"/>
+		</visual>
+	</link>
+	<joint name="right_wheel_joint" type="continuous">
+		<parent link="base_link"/>
+		<child link="right_wheel"/>
+		<origin xyz="0 -0.1375 0" rpy="${pi/2} 0 0"/>
+		<axis xyz="0 0 -1"/>
+	</joint>
+	<link name="right_wheel">
+		<visual>
+			<geometry>
+				<cylinder length="0.01" radius="0.045" />/>
+			</geometry>
+			<material name="blue"/>
+		</visual>
+	</link>
 </robot>

Commit message: Finish Urdf

File: description/robot_core.xacro (robot description, xacro)
@@ -1,3 +1,4 @@
 <?xml version="1.0"?>
+<xacro:include filename="inertial_macros.xacro" />
 <robot xmlns:xacro="http://www.ros.org/wiki/xacro">
 	<material name="white">
@@ -28,4 +29,10 @@
 		    <material name="white"/>
 		</visual>
+		<collision>
+			<origin xyz="0 0 0.03915" rpy="0 0 0"/>
+		    <geometry>
+		        <box size="0.25 0.25 0.12"/>
+		    </geometry>
+		</collision>
 	</link>
 	<joint name="left_wheel_joint" type="continuous">
@@ -42,4 +49,9 @@
 			<material name="blue"/>
 		</visual>
+		<collision>
+			<geometry>
+				<cylinder length="0.01" radius="0.045" />/>
+			</geometry>
+		</collision>
 	</link>
 	<joint name="right_wheel_joint" type="continuous">
@@ -56,4 +68,45 @@
 			<material name="blue"/>
 		</visual>
+		<collision>
+			<geometry>
+				<cylinder length="0.01" radius="0.045" />/>
+			</geometry>
+		</collision>
+	</link>
+	<joint name="front_caster_wheel_joint" type="fixed">
+		<parent link="chassis"/>
+		<child link="front_caster_wheel"/>
+		<origin xyz="0.075 0 -0.02085" rpy="0 0 0"/>
+	</joint>
+	<link name="front_caster_wheel">
+		<visual>
+			<geometry>
+				<sphere radius="0.0228125"/>
+			</geometry>
+			<material name="black"/>
+		</visual>
+		<collision>
+			<geometry>
+				<sphere radius="0.0228125"/>
+			</geometry>
+		</collision>
+	</link>
+	<joint name="back_caster_wheel_joint" type="fixed">
+		<parent link="chassis"/>
+		<child link="back_caster_wheel"/>
+		<origin xyz="-0.075 0 -0.02085" rpy="0 0 0"/>
+	</joint>
+	<link name="back_caster_wheel">
+		<visual>
+			<geometry>
+				<sphere radius="0.0228125"/>
+			</geometry>
+			<material name="black"/>
+		</visual>
+		<collision>
+			<geometry>
+				<sphere radius="0.0228125"/>
+			</geometry>
+		</collision>
 	</link>
 </robot>

Commit message: Update Urdf

File: description/robot_core.xacro (robot description, xacro)
@@ -1,5 +1,5 @@
 <?xml version="1.0"?>
-<xacro:include filename="inertial_macros.xacro" />
 <robot xmlns:xacro="http://www.ros.org/wiki/xacro">
+	<xacro:include filename="inertial_macros.xacro" />
 	<material name="white">
 	    <color rgba="1 1 1 1"/>
@@ -14,6 +14,7 @@
 	    <color rgba="0 0 0 1"/>
 	</material>
-	<link name="base_link">
-	</link>
+	<!-- BASE LINK -->
+	<link name="base_link"></link>
+	<!-- CHASSIS -->
 	<joint name="chassis_joint" type="fixed">
 		<parent link="base_link"/>
@@ -35,5 +36,12 @@
 		    </geometry>
 		</collision>
+		<xacro:inertial_box mass="0.5" x="0.25" y="0.25" z="0.12">
+			<origin xyz="0 0 0.03915" rpy="0 0 0"/>
+		</xacro:inertial_box>
 	</link>
+	<gazebo reference="chassis">
+		<material>Gazebo/White</material>
+	</gazebo>
+	<!-- LEFT WHEEL -->
 	<joint name="left_wheel_joint" type="continuous">
 		<parent link="base_link"/>
@@ -54,5 +62,12 @@
 			</geometry>
 		</collision>
+		<xacro:inertial_cylinder mass="0.1" length="0.01" radius="0.045">
+			<origin xyz="0 0 0" rpy="0 0 0"/>
+		</xacro:inertial_cylinder>
 	</link>
+	<gazebo reference="left_wheel">
+    	<material>Gazebo/Blue</material>
+	</gazebo>
+	<!-- RIGHT WHEEL -->
 	<joint name="right_wheel_joint" type="continuous">
 		<parent link="base_link"/>
@@ -73,5 +88,12 @@
 			</geometry>
 		</collision>
+		<xacro:inertial_cylinder mass="0.1" length="0.01" radius="0.045">
+			<origin xyz="0 0 0" rpy="0 0 0"/>
+		</xacro:inertial_cylinder>
 	</link>
+	<gazebo reference="right_wheel">
+    	<material>Gazebo/Blue</material>
+	</gazebo>
+	<!-- FRONT CASTER -->
 	<joint name="front_caster_wheel_joint" type="fixed">
 		<parent link="chassis"/>
@@ -82,5 +104,5 @@
 		<visual>
 			<geometry>
-				<sphere radius="0.0228125"/>
+				<sphere radius="0.02415"/>
 			</geometry>
 			<material name="black"/>
@@ -88,8 +110,17 @@
 		<collision>
 			<geometry>
-				<sphere radius="0.0228125"/>
+				<sphere radius="0.02415"/>
 			</geometry>
 		</collision>
+		<xacro:inertial_sphere mass="0.1" radius="0.02415">
+			<origin xyz="0 0 0" rpy="0 0 0"/>
+		</xacro:inertial_sphere>
+		<gazebo reference="caster_wheel">
+			<material>Gazebo/Black</material>
+			<mu1 value="0.001"/>
+			<mu2 value="0.001"/>
+		</gazebo>
 	</link>
+	<!-- BACK CASTER -->
 	<joint name="back_caster_wheel_joint" type="fixed">
 		<parent link="chassis"/>
@@ -100,5 +131,5 @@
 		<visual>
 			<geometry>
-				<sphere radius="0.0228125"/>
+				<sphere radius="0.02415"/>
 			</geometry>
 			<material name="black"/>
@@ -106,7 +137,15 @@
 		<collision>
 			<geometry>
-				<sphere radius="0.0228125"/>
+				<sphere radius="0.02415"/>
 			</geometry>
 		</collision>
+		<xacro:inertial_sphere mass="0.1" radius="0.02415">
+			<origin xyz="0 0 0" rpy="0 0 0"/>
+		</xacro:inertial_sphere>
 	</link>
+	<gazebo reference="caster_wheel">
+		<material>Gazebo/Black</material>
+		<mu1 value="0.001"/>
+		<mu2 value="0.001"/>
+	</gazebo>
 </robot>

Commit message: Bugfix

File: description/robot_core.xacro (robot description, xacro)
@@ -53,5 +53,5 @@
 		<visual>
 			<geometry>
-				<cylinder length="0.01" radius="0.045" />/>
+				<cylinder length="0.01" radius="0.045" />
 			</geometry>
 			<material name="blue"/>
@@ -59,5 +59,5 @@
 		<collision>
 			<geometry>
-				<cylinder length="0.01" radius="0.045" />/>
+				<cylinder length="0.01" radius="0.045" />
 			</geometry>
 		</collision>

Commit message: Bugfix

File: description/robot_core.xacro (robot description, xacro)
@@ -79,5 +79,5 @@
 		<visual>
 			<geometry>
-				<cylinder length="0.01" radius="0.045" />/>
+				<cylinder length="0.01" radius="0.045" />
 			</geometry>
 			<material name="blue"/>
@@ -85,5 +85,5 @@
 		<collision>
 			<geometry>
-				<cylinder length="0.01" radius="0.045" />/>
+				<cylinder length="0.01" radius="0.045" />
 			</geometry>
 		</collision>

Commit message: Update robot model

File: description/robot_core.xacro (robot description, xacro)
@@ -1,4 +1,17 @@
 <?xml version="1.0"?>
 <robot xmlns:xacro="http://www.ros.org/wiki/xacro">
+	 <xacro:property name="chassis_length" value="0.2"/>
+    <xacro:property name="chassis_width" value="0.2"/>
+    <xacro:property name="chassis_height" value="0.01"/>
+    <xacro:property name="chassis_mass" value="1.0"/>
+	<xacro:property name="chassis_base_offset" value='0.1'>
+    <xacro:property name="wheel_radius" value="0.045"/>
+    <xacro:property name="wheel_thickness" value="0.01"/>
+    <xacro:property name="wheel_mass" value="0.05"/>
+    <xacro:property name="wheel_offset" value="0.0925"/>
+    <xacro:property name="caster_wheel_radius" value="wheel_radius-chassis base_offset"/>
+    <xacro:property name="caster_wheel_mass" value="0.01"/>
+    <xacro:property name="caster_wheel_offset_x" value="0.075"/>
+    <xacro:property name="caster_wheel_offset_z" value="${-chassis_base_offset}"/>
 	<xacro:include filename="inertial_macros.xacro" />
 	<material name="white">
@@ -32,18 +45,18 @@
 	<link name="chassis">
 		<visual>
-			<origin xyz="0 0 0.03915" rpy="0 0 0" />
+			<origin yz="0 0 ${chassis_height/2 - chassis_base_offset}" rpy="0 0 0" />
 			<geometry>
-				<box size="0.25 0.25 0.12" />
+				 <box size="${chassis_length} ${chassis_width} ${chassis_height}"/>
 			</geometry>
 			<material name="white" />
 		</visual>
 		<collision>
-			<origin xyz="0 0 0.03915" rpy="0 0 0" />
+			<origin yz="0 0 ${chassis_height/2 - chassis_base_offset}" rpy="0 0 0" />
 			<geometry>
-				<box size="0.25 0.25 0.12" />
+				 <box size="${chassis_length} ${chassis_width} ${chassis_height}"/>
 			</geometry>
 		</collision>
 		<xacro:inertial_box mass="0.5" x="0.25" y="0.25" z="0.12">
-			<origin xyz="0 0 0.03915" rpy="0 0 0" />
+			<origin xyz="0 0 ${chassis_height/2 - chassis_base_offset}" rpy="0 0 0" />
 		</xacro:inertial_box>
 	</link>
@@ -57,5 +70,5 @@
 		<parent link="base_link" />
 		<child link="left_wheel" />
-		<origin xyz="0 0.1375 0" rpy="-${pi/2} 0 0" />
+		<origin xyz="0 ${wheel_offset} 0" rpy="-${pi/2} 0 0" />
 		<axis xyz="0 0 1" />
 	</joint>
@@ -63,5 +76,5 @@
 		<visual>
 			<geometry>
-				<cylinder length="0.01" radius="0.045" />
+				<cylinder length="${wheel_thickness}" radius="${wheel_radius}" />
 			</geometry>
 			<material name="blue" />
@@ -69,8 +82,8 @@
 		<collision>
 			<geometry>
-				<sphere radius="0.045" />
+				<sphere radius="${wheel_radius}" />
 			</geometry>
 		</collision>
-		<xacro:inertial_cylinder mass="0.1" length="0.01" radius="0.045">
+		<xacro:inertial_cylinder mass="${wheel_mass}" length="${wheel_thickness}" radius="${wheel_radius}">
 			<origin xyz="0 0 0" rpy="0 0 0" />
 		</xacro:inertial_cylinder>
@@ -85,5 +98,5 @@
 		<parent link="base_link" />
 		<child link="right_wheel" />
-		<origin xyz="0 -0.1375 0" rpy="${pi/2} 0 0" />
+		<origin xyz="0 ${-wheel_offset} 0" rpy="${pi/2} 0 0" />
 		<axis xyz="0 0 -1" />
 	</joint>
@@ -91,5 +104,5 @@
 		<visual>
 			<geometry>
-				<cylinder length="0.01" radius="0.045" />
+				<cylinder length="${wheel_thickness}" radius="${wheel_radius}" />
 			</geometry>
 			<material name="blue" />
@@ -97,8 +110,8 @@
 		<collision>
 			<geometry>
-				<sphere radius="0.045" />
+				<sphere radius="${wheel_radius}"/>
 			</geometry>
 		</collision>
-		<xacro:inertial_cylinder mass="0.1" length="0.01" radius="0.045">
+		<xacro:inertial_cylinder mass="${wheel_mass}" length="${wheel_thickness}" radius="${wheel_radius}">
 			<origin xyz="0 0 0" rpy="0 0 0" />
 		</xacro:inertial_cylinder>
@@ -113,10 +126,10 @@
 		<parent link="chassis" />
 		<child link="front_caster_wheel" />
-		<origin xyz="0.075 0 -0.02085" rpy="0 0 0" />
+		<origin xyz="${caster_offset_x} 0 ${caster_offset_z}" rpy="0 0 0" />
 	</joint>
 	<link name="front_caster_wheel">
 		<visual>
 			<geometry>
-				<sphere radius="0.02415" />
+				<sphere radius="${caster_radius}" />
 			</geometry>
 			<material name="black" />
@@ -124,8 +137,8 @@
 		<collision>
 			<geometry>
-				<sphere radius="0.02415" />
-			</geometry>
+				<sphere radius="${caster_radius}"  />
+			</geometry>r
 		</collision>
-		<xacro:inertial_sphere mass="0.1" radius="0.02415">
+		<xacro:inertial_sphere mass="0.1" radius="${caster_radius}">
 			<origin xyz="0 0 0" rpy="0 0 0"/>
 		</xacro:inertial_sphere>
@@ -142,10 +155,10 @@
 		<parent link="chassis" />
 		<child link="back_caster_wheel" />
-		<origin xyz="-0.075 0 -0.02085" rpy="0 0 0" />
+		<origin xyz="${-caster_offset_x} 0 ${caster_offset_z}" rpy="0 0 0" />
 	</joint>
 	<link name="back_caster_wheel">
 		<visual>
 			<geometry>
-				<sphere radius="0.02415" />
+				<sphere radius="${caster_radius}" />
 			</geometry>
 			<material name="black" />
@@ -153,8 +166,8 @@
 		<collision>
 			<geometry>
-				<sphere radius="0.02415" />
+				<sphere radius="${caster_radius}" />
 			</geometry>
 		</collision>
-		<xacro:inertial_sphere mass="0.1" radius="0.02415">
+		<xacro:inertial_sphere mass="0.1" radius="${caster_radius}">
 			<origin xyz="0 0 0" rpy="0 0 0"/>
 		</xacro:inertial_sphere>

Commit message: Fully updated robot_core_config

File: description/robot_core.xacro (robot description, xacro)
@@ -1,5 +1,5 @@
 <?xml version="1.0"?>
 <robot xmlns:xacro="http://www.ros.org/wiki/xacro">
-	 <xacro:property name="chassis_length" value="0.2"/>
+	<xacro:property name="chassis_length" value="0.2"/>
     <xacro:property name="chassis_width" value="0.2"/>
     <xacro:property name="chassis_height" value="0.01"/>
@@ -138,5 +138,5 @@
 			<geometry>
 				<sphere radius="${caster_radius}"  />
-			</geometry>r
+			</geometry>
 		</collision>
 		<xacro:inertial_sphere mass="0.1" radius="${caster_radius}">
